Commit message: fixed rotation of linear velocity and threshold filter for small target velocities

File: multi_robot_launcher/urdf/caster_wheel.xacro (robot description, xacro)
@@ -59,8 +59,8 @@
                 <xacro:insert_block name="material_dark_grey" />
             </visual>
-            <collision>
+            <collision  >
                 <origin xyz="0 0 0" rpy="0 0 0" />
                 <geometry>
-                <mesh filename="package://mir_description/meshes/visual/wheel.stl" />
+                    <mesh filename="package://mir_description/meshes/visual/wheel.stl" />
                 </geometry>
             </collision>

Commit message: Fixed caster wheels xacro

File: multi_robot_launcher/urdf/caster_wheel.xacro (robot description, xacro)
@@ -1,8 +1,8 @@
 <?xml version="1.0"?>
 <robot xmlns:xacro="http://ros.org/wiki/xacro">
-    <xacro:macro name="caster_wheel" params="prefix locationprefix locationright damping_steering friction_steering damping_wheel friction_wheel">
+    <xacro:macro name="caster_wheel" params="prefix locationprefix locationright wheel_base_dx damping_steering friction_steering damping_wheel friction_wheel">
         <!-- caster hub -->
         <joint name="${prefix}${locationprefix}_caster_rotation_joint" type="continuous">
-            <origin xyz="${mir_200_front_caster_wheel_base_dx} ${-mir_200_caster_wheel_base_dy * locationright} ${mir_200_caster_wheel_base_dz}" rpy="0 0 0" />
+            <origin xyz="${wheel_base_dx} ${-mir_200_caster_wheel_base_dy * locationright} ${mir_200_caster_wheel_base_dz}" rpy="0 0 0" />
             <parent link="${prefix}base_link" />
             <child link="${prefix}${locationprefix}_caster_rotation_link" />

File: multi_robot_launcher/urdf/mir200.xacro (robot description, xacro)
@@ -58,10 +58,10 @@
     </gazebo>
     <!-- wheels -->
-    <xacro:actuated_wheel prefix="${prefix}" locationprefix="left" locationright="-1" damping_wheel="0.0" friction_wheel="0.0"/>
+    <xacro:actuated_wheel prefix="${prefix}" locationprefix="left"  locationright="-1" damping_wheel="0.0" friction_wheel="0.0"/>
     <xacro:actuated_wheel prefix="${prefix}" locationprefix="right" locationright="1" damping_wheel="0.0" friction_wheel="0.0"/>
-    <xacro:caster_wheel prefix="${prefix}" locationprefix="fl" locationright="-1" damping_steering="0.0" friction_steering="0.0" damping_wheel="0.0" friction_wheel="0.0"/>
-    <xacro:caster_wheel prefix="${prefix}" locationprefix="fr" locationright="1"  damping_steering="0.0" friction_steering="0.0" damping_wheel="0.0" friction_wheel="0.0"/>
-    <xacro:caster_wheel prefix="${prefix}" locationprefix="bl" locationright="-1" damping_steering="0.0" friction_steering="0.0" damping_wheel="0.0" friction_wheel="0.0"/>
-    <xacro:caster_wheel prefix="${prefix}" locationprefix="br" locationright="1"  damping_steering="0.0" friction_steering="0.0" damping_wheel="0.0" friction_wheel="0.0"/>
+    <xacro:caster_wheel prefix="${prefix}" locationprefix="fl" locationright="-1"   wheel_base_dx="${mir_200_front_caster_wheel_base_dx}" damping_steering="0.0" friction_steering="0.0" damping_wheel="0.0" friction_wheel="0.0"/>
+    <xacro:caster_wheel prefix="${prefix}" locationprefix="fr" locationright="1"    wheel_base_dx="${mir_200_front_caster_wheel_base_dx}" damping_steering="0.0" friction_steering="0.0" damping_wheel="0.0" friction_wheel="0.0"/>
+    <xacro:caster_wheel prefix="${prefix}" locationprefix="bl" locationright="-1"   wheel_base_dx="${mir_200_back_caster_wheel_base_dx}" damping_steering="0.0" friction_steering="0.0" damping_wheel="0.0" friction_wheel="0.0"/>
+    <xacro:caster_wheel prefix="${prefix}" locationprefix="br" locationright="1"    wheel_base_dx="${mir_200_back_caster_wheel_base_dx}" damping_steering="0.0" friction_steering="0.0" damping_wheel="0.0" friction_wheel="0.0"/>
     <!-- IMU -->
     <joint name="${prefix}base_link_to_imu_joint" type="fixed">
@@ -107,5 +107,6 @@
     </joint>
     <link name="${prefix}us_2_frame" />
-    <!-- <joint name="${prefix}base_link_surface_joint" type="fixed">
+    <!-- Ultrasound sensor plugin missing ?! -->
+    <joint name="${prefix}base_link_surface_joint" type="fixed">
       <origin xyz="${mir_200_act_wheel_dx} 0 0.352" rpy="0 0 0" />
       <parent link="${prefix}base_link" />
@@ -113,5 +114,5 @@
       <axis xyz="0 0 1" />
     </joint>
-    <link name="${prefix}surface"/> -->
+    <link name="${prefix}surface"/>
     <xacro:mir_200_wheel_transmissions prefix="${prefix}"/>
     <!-- disabled, because it doesn't make a difference in Gazebo: -->
