Commit message: added sapwn trubine urdf

File: multi_robot_launcher/urdf/objects/turbine.urdf.xacro (robot description, xacro)
@@ -4,17 +4,17 @@
         <link name="${link_name}">
             <inertial>
-                <origin xyz="-2.0 -1.0 0.0" rpy="1.57 0.0 1.57" />
+                <origin xyz="0.0 0 0.0" rpy="0 0.0 0" />
                 <mass value="1"/>
                 <inertia ixx="1.0" ixy="0.0" ixz="0.0" iyy="1.0" iyz="0.0" izz="1.0"/>
             </inertial>
             <visual>
-                <origin xyz="-2.0 -1.0 0.0" rpy="1.57 0.0 1.57" />
+                <origin xyz="-0.0 0 0.1" rpy="0 0.0 0" />
                 <geometry>
-                    <mesh filename="package://multi_robot_launcher/urdf/meshes/Mcqueen_Car.stl" scale="0.025 0.025 0.025"/>
+                    <mesh filename="package://multi_robot_launcher/urdf/meshes/Turbine.stl" scale="0.07 0.07 0.07"/>
                 </geometry>
             </visual>
         </link>
         <gazebo reference="${link_name}">
-            <material>Gazebo/Orange</material>
+            <material>Gazebo/Grey</material>
         </gazebo>
     </xacro:macro>

File: multi_robot_launcher/urdf/transport_object.urdf.xacro (robot description, xacro)
@@ -12,5 +12,5 @@
     <xacro:arg name="z_size" default="" />
     <xacro:macro name="transport_object" params="object_name x y z x_size y_size z_size">
-        <xacro:include filename="$(find multi_robot_launcher)/urdf/objects/${object_name}.xacro"/>
+        <xacro:include filename="$(find multi_robot_launcher)/urdf/objects/${object_name}.urdf.xacro"/>
         <link name="plate_link">
             <inertial>
