Commit message: Changed car properties

File: multi_robot_launcher/urdf/objects/car.urdf.xacro (robot description, xacro)
@@ -4,10 +4,10 @@
         <link name="${link_name}">
             <inertial>
-                <origin xyz="-2.0 -1.0 0.0" rpy="1.57 0.0 1.57" />
+                <origin xyz="0 -0. 0.0" rpy="1.57 0.0 1.57" />
                 <mass value="1"/>
                 <inertia ixx="1.0" ixy="0.0" ixz="0.0" iyy="1.0" iyz="0.0" izz="1.0"/>
             </inertial>
             <visual>
-                <origin xyz="-2.0 -1.0 0.0" rpy="1.57 0.0 1.57" />
+                <origin xyz="-2.0 -0.9 0.0" rpy="1.57 0.0 1.57" />
                 <geometry>
                     <mesh filename="package://multi_robot_launcher/urdf/meshes/Mcqueen_Car.stl" scale="0.025 0.025 0.025"/>
@@ -16,5 +16,4 @@
         </link>
         <gazebo reference="${link_name}">
-            <material>Gazebo/Orange</material>
         </gazebo>
     </xacro:macro>

Commit message: Changed Translport launch files

File: multi_robot_launcher/urdf/objects/car.urdf.xacro (robot description, xacro)
@@ -9,5 +9,5 @@
             </inertial>
             <visual>
-                <origin xyz="-2.0 -1.0 0.0" rpy="1.57 0.0 1.57" />
+                <origin xyz="-2.0 -0.9 0.0" rpy="1.57 0.0 1.57" />
                 <geometry>
                     <mesh filename="package://multi_robot_launcher/urdf/meshes/Mcqueen_Car.stl" scale="0.025 0.025 0.025"/>
@@ -16,5 +16,4 @@
         </link>
         <gazebo reference="${link_name}">
-            <material>Gazebo/Orange</material>
         </gazebo>
     </xacro:macro>

Commit message: Modified transport objects

File: multi_robot_launcher/urdf/objects/car.urdf.xacro (robot description, xacro)
@@ -11,5 +11,5 @@
                 <origin xyz="-2.0 -0.9 0.0" rpy="1.57 0.0 1.57" />
                 <geometry>
-                    <mesh filename="package://multi_robot_launcher/urdf/meshes/Mcqueen_Car.stl" scale="0.025 0.025 0.025"/>
+                    <mesh filename="package://multi_robot_launcher/urdf/meshes/car.stl" scale="0.025 0.025 0.025"/>
                 </geometry>
             </visual>

File: multi_robot_launcher/urdf/objects/rib.urdf.xacro (robot description, xacro)
@@ -11,5 +11,5 @@
                 <origin xyz="0.1 -4.0 0.075" rpy="0 0.0 1.57" />
                 <geometry>
-                    <mesh filename="package://multi_robot_launcher/urdf/meshes/Rib.stl" scale="0.01 0.01 0.01"/>
+                    <mesh filename="package://multi_robot_launcher/urdf/meshes/rib.stl" scale="0.01 0.01 0.01"/>
                 </geometry>
             </visual>
